File: Projects/Antifurto/TILT - PIC/Tilt-PIC12F635 + 4N35.brd (EAGLE design)
At the start: 100 x 80 mm, 15 parts

Commit message: 2015-02-06 07:54 - commit with no comment
Parts:
- removed MM1, MM2: MAMMUTH03, Ln-Varie:MAMMUTH03
- removed U$3: JUMPER2X1, Ln-Varie:SIP02
- added *OCT, PWR: MAMMUTH03, Ln-Varie:MAMMUTH03
- added ALRM, JLED: JUMPER2X1, Ln-Varie:SIP02
- moved OK1 30.5 mm to (45.7, 29.2), turned to 270 degrees
- moved R5 26.7 mm to (50.8, 36.8), turned to 180 degrees
- moved LED1 24.2 mm to (38.1, 43.2), turned to 90 degrees
- moved R4 23.7 mm to (25.4, 26.7), turned to 270 degrees
- moved D1 21.6 mm to (49.5, 39.4)
- moved R3 20.7 mm to (31.8, 38.1), turned to 0 degrees
- moved C1 16.2 mm to (36.8, 21.6), turned to 90 degrees
- moved R1 14.5 mm to (17.8, 27.9), turned to 270 degrees
- moved U$1 10.5 mm to (19.1, 44.5)
- moved TILT 10.2 mm to (41.9, 21.6), turned to 180 degrees
- moved R2 4.58 mm to (21.6, 27.9)
- renumbered U$2 to UP1
Connections:
- removed net N$5: U$3.1, UP1.3
- new net N$4: C1.2, UP1.5
- net +12V: now also ALRM.1
- net +5V: now also PWR.P$3
- net GND: now also PWR.P$1; no longer C1.1, MM2.P$1
- net ICSPDAT: now also JLED.1
- net N$3: no longer MM2.P$3
- net N$6: now also JLED.2; no longer U$3.2
- net TILT: now also C1.1; no longer UP1.5
- net TO_ALARM: now also ALRM.2
- net VSS: no longer MM1.P$1
